File: FinalSchematic.kicad_sch (KiCad schematic)
At the start: 49 parts, among them IC1 SC-1020, J1 RF_Ant, J14 RX_Output, J2 Conn_01x08_Pin, J3 Conn_01x02_Pin, J6 TX_Input

Commit message: Notes and Minor Tweaks
Connections:
- net T8: now reaches C6.2, IC1.3 (VBB), J2.3 (Pin_3), R2.1, TP6.1
- net PowerMeter: now reaches C18.1, C21.1, J2.1 (Pin_1), R5.1, TP7.1
- net PAV: now reaches C4.1, C5.1, IC1.4 (VCC2), J2.4 (Pin_4), R1.2, TP4.1
Changed lines of the file:
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@@
 	(generator_version "9.0")
 	(paper "A4")
+	(text_box "NOTE\n\nSome connector names are not exactly how they might be listed in the original schematics"
+		(exclude_from_sim no)
+		(at 16.51 167.64 0)
+		(size 58.42 22.86)
+		(margins 0.9525 0.9525 0.9525 0.9525)
+		(stroke
+			(width 0)
+			(type solid)
+		)
+		(fill
+			(type none)
+		)
+		(effects
+			(font
+				(size 1.27 1.27)
+			)
+			(justify left top)
+		)
+	)
+	(text_box "From Service Manual - Section 5-1-1 Antenna Switching Circuit (PA Unit)\n\nRecieve signals from the PA UNIT antenna connector (J1) pass to the antenna switching circuit (D1,D2) via the PA UNIT low-pass filter consisting of L2 through L5, C9, C10 and C12 through C17. While receiving, approximately 13.8 volts is applied to the cathode side of D2 thus causing D2 to be reverse-biased and switched OFF. While transmitting, T8V is supplied to D2 from D1 which causes D2 to switch ON. D2 and C11 ground any leakage to protect the receiver.\n\nIn addition, because the anode side of D1 is at ground level during reception, D1 is reverse-biased and switched OFF, providing good isolation from IC1. While transmitting, T8V keeps D1 turned ON. Thr receive signals feed via P2 to the RF-YGR UNIT(J4)\n"
+		(exclude_from_sim no)
+		(at 218.44 15.24 0)
+		(size 59.69 38.1)
+		(margins 0.9525 0.9525 0.9525 0.9525)
+		(stroke
+			(width 0)
+			(type solid)
+		)
+		(fill
+			(type none)
+		)
+		(effects
+			(font
+				(size 1.27 1.27)
+			)
+			(justify left top)
+		)
+	)
 	(junction
 		(at 220.98 97.79)
@@
 		)
 	)
+	(global_label "PAV"
+		(shape input)
+		(at 157.48 45.72 180)
+		(fields_autoplaced yes)
+		(effects
+			(font
+				(size 1.27 1.27)
+			)
+			(justify right)
+		)
+		(property "Intersheetrefs" "${INTERSHEET_REFS}"
+			(at 151.0476 45.72 0)
+			(effects
+				(font
+					(size 1.27 1.27)
+				)
+				(justify right)
+				(hide yes)
+			)
+		)
+	)
+	(global_label "PowerMeter"
+		(shape input)
+		(at 240.03 58.42 0)
+		(fields_autoplaced yes)
+		(effects
+			(font
+				(size 1.27 1.27)
+			)
+			(justify left)
+		)
+		(property "Intersheetrefs" "${INTERSHEET_REFS}"
+			(at 253.78 58.42 0)
+			(effects
+				(font
+					(size 1.27 1.27)
+				)
+				(justify left)
+				(hide yes)
+			)
+		)
+	)
+	(global_label "T8"
+		(shape input)
+		(at 176.53 55.88 0)
+		(fields_autoplaced yes)
+		(effects
+			(font
+				(size 1.27 1.27)
+			)
+			(justify left)
+		)
+		(property "Intersheetrefs" "${INTERSHEET_REFS}"
+			(at 181.6923 55.88 0)
+			(effects
+				(font
+					(size 1.27 1.27)
+				)
+				(justify left)
+				(hide yes)
+			)
+		)
+	)
