File: PA_UNIT.kicad_sch (KiCad schematic)
At the start: 49 parts, among them IC1 SC-1020, J1 RF_Ant, J14 RX_Output, J2 Conn_01x08_Pin, J3 Conn_01x02_Pin, J6 TX_Input

Commit message: Tranmitter Notes from Service manual
Other:
- note added: "a"
- moved on the sheet: C19, C20, D4
